Commit message: fix: enhance error handling in Loader and update URDF model paths (Fixes #48)

File: tests/models/UR5/UR5.urdf (robot description, URDF)
Before this commit: robot ur5_robot, 11 links, 10 joints
Links:
- link base_link_inertia: geometry collision mesh filename=base.stl; visual mesh filename=base.stl
- link forearm_link: geometry collision mesh filename=forearm.stl; visual mesh filename=forearm.stl
- link shoulder_link: geometry collision mesh filename=shoulder.stl; visual mesh filename=shoulder.stl
- link upper_arm_link: geometry collision mesh filename=upperarm.stl; visual mesh filename=upperarm.stl
- link wrist_1_link: geometry collision mesh filename=wrist1.stl; visual mesh filename=wrist1.stl
- link wrist_2_link: geometry collision mesh filename=wrist2.stl; visual mesh filename=wrist2.stl
- link wrist_3_link: geometry collision mesh filename=wrist3.stl; visual mesh filename=wrist3.stl
